Commit message: carry smach completed

File: src/Hardware/robotino/robotino_description/urdf/robotino_armful.urdf.xacro (robot description, xacro)
@@ -1,132 +1,36 @@
-<robot xmlns:xacro="http://www.ros.org/wiki/xacro" name="robotino">
-  <!-- ==================== Includes ==================== -->
-  <xacro:include filename="$(find xarm_description)/urdf/xarm6/xarm6.urdf.xacro" />
-  <xacro:include filename="$(find xarm_description)/urdf/xarm_device_macro.xacro" />
-  <!-- ==================== Properties ==================== -->
-  <xacro:property name="mesh_scale" value="0.01 0.01 0.01"/>
-  <xacro:property name="wheel_mesh" value="package://robotino_description/model/Robotino3_SplitWheel.dae"/>
-  <xacro:property name="body_mesh" value="package://robotino_description/model/Robotino3_SplitMain_NoCamera.dae"/>
-  <xacro:property name="tower_mesh" value="package://robotino_description/model/Robotino3_Platform-xarm.dae"/>
-  <xacro:property name="hokuyo_mesh" value="package://robotino_description/meshes/sensors/hokuyo.dae"/>
-  <xacro:property name="kinect_mesh" value="package://robotino_description/meshes/sensors/kinect.dae"/>
-  <!-- ==================== Macros ==================== -->
-  <xacro:macro name="wheel_link" params="index xyz rpy">
-    <link name="wheel${index}_link">
-      <inertial>
-        <mass value="1.0"/>
-        <origin xyz="0 0 0" rpy="0 0 0"/>
-        <inertia ixx="0.01" iyy="0.01" izz="0.01" ixy="0" ixz="0" iyz="0"/>
-      </inertial>
-      <visual>
-        <origin xyz="0 0 0" rpy="0 0 0"/>
-        <geometry>
-          <mesh filename="${wheel_mesh}" scale="${mesh_scale}"/>
-        </geometry>
-      </visual>
-      <collision>
-        <origin xyz="0 0 0" rpy="0 0 0"/>
-        <geometry>
-          <mesh filename="${wheel_mesh}" scale="${mesh_scale}"/>
-        </geometry>
-      </collision>
-    </link>
-    <joint name="wheel${index}_joint" type="continuous">
-      <parent link="base_link"/>
-      <child link="wheel${index}_link"/>
-      <origin xyz="${xyz}" rpy="${rpy}"/>
-      <axis xyz="0 1 0"/>
-    </joint>
-  </xacro:macro>
-  <!-- ==================== Base ==================== -->
-  <link name="base_link">
-    <inertial>
-      <origin xyz="0 0 0.03" rpy="0 0 0"/>
-      <mass value="35.0"/>
-      <inertia ixx="1.0" iyy="1.0" izz="1.0" ixy="0.0" ixz="0.0" iyz="0.0"/>
-    </inertial>
-    <visual>
-      <origin xyz="0 0 0.035" rpy="0 0 1.5707"/>
-      <geometry>
-        <mesh filename="${body_mesh}" scale="${mesh_scale}"/>
-      </geometry>
-    </visual>
-    <collision>
-      <origin xyz="0 0 0.035" rpy="0 0 1.5707"/>
-      <geometry>
-        <mesh filename="${body_mesh}" scale="${mesh_scale}"/>
-      </geometry>
-    </collision>
-    <collision>
-      <origin xyz="0 0 0.03" rpy="0 0 0"/>
-      <geometry>
-        <box size="0.4 0.4 0.06"/>
-      </geometry>
-    </collision>
-  </link>
-  <!-- ==================== Wheels ==================== -->
-  <xacro:wheel_link index="0" xyz="-0.1825 -0.0001 0.059154" rpy="0 0 1.570796"/>
-  <xacro:wheel_link index="1" xyz="0.090625 -0.157067 0.059154" rpy="0 0 3.665191"/>
-  <xacro:wheel_link index="2" xyz="0.090625 0.156867 0.059154" rpy="0 0 -0.523599"/>
-  <!-- ==================== Tower (Platform) ==================== -->
-  <link name="platform_link">
-    <visual>
-      <origin xyz="0 0 -0.70" rpy="0 0 1.5707"/>
-      <geometry>
-        <mesh filename="${tower_mesh}" scale="0.009 0.009 0.009"/>
-      </geometry>
-    </visual>
-    <collision>
-      <origin xyz="0 0 -0.70" rpy="0 0 1.5707"/>
-      <geometry>
-        <mesh filename="${tower_mesh}" scale="0.009 0.009 0.009"/>
-      </geometry>
-    </collision>
-  </link>
-  <joint name="platform_joint" type="fixed">
+<?xml version="1.0"?>
+<robot name="festoshi" xmlns:xacro="http://ros.org/wiki/xacro">
+  <!-- ARGUMENTS -->
+  <xacro:arg name="add_gripper" default="false"/>
+  <xacro:arg name="add_vacuum_gripper" default="false"/>
+  <xacro:arg name="effort_control" default="true"/>
+  <xacro:arg name="xarm_velocity_control" default="false"/>
+  <xacro:arg name="model1300" default="false"/>
+  <xacro:arg name="add_realsense_d435i" default="false"/>
+  <xacro:arg name="add_d435i_links" default="false"/>
+  <xacro:arg name="robot_sn" default=""/>
+  <xacro:arg name="namespace" default=""/>
+  <!-- INCLUDE base first, which is a full robot -->
+  <xacro:include filename="$(find robotino_description)/urdf/robotino_armless.urdf.xacro"/>
+  <!-- INCLUDE arm, which defines a macro -->
+  <xacro:include filename="$(find xarm_description)/urdf/xarm_device.urdf.xacro"/>
+  <!-- Instantiate xarm_device directly -->
+  <xacro:xarm_device
+    robot_type="xarm"
+    dof="5"
+    add_gripper="$(arg add_gripper)"
+    add_vacuum_gripper="$(arg add_vacuum_gripper)"
+    effort_control="$(arg effort_control)"
+    velocity_control="$(arg xarm_velocity_control)"
+    model1300="$(arg model1300)"
+    add_realsense_d435i="$(arg add_realsense_d435i)"
+    add_d435i_links="$(arg add_d435i_links)"
+    robot_sn="$(arg robot_sn)"
+    hw_ns="$(arg namespace)" />
+  <!-- Connect base and arm -->
+  <joint name="xarm_mount" type="fixed">
     <parent link="base_link"/>
-    <child link="platform_link"/>
-    <origin xyz="0 0 0.455" rpy="0 0 0"/>
+    <child link="link_base"/>
+    <origin xyz="0 0 0.75" rpy="0 0 0"/>
   </joint>
-  <!-- ==================== Kinect Sensor ==================== -->
-  <link name="camera_link">
-    <visual>
-      <origin xyz="0.15 0 0" rpy="0 0 1.57"/>
-      <geometry>
-        <mesh filename="${kinect_mesh}" scale="1 1 1"/>
-      </geometry>
-    </visual>
-    <collision>
-      <origin xyz="0.15 0 0" rpy="0 0 1.57"/>
-      <geometry>
-        <mesh filename="${kinect_mesh}" scale="1 1 1"/>
-      </geometry>
-    </collision>
-  </link>
-  <joint name="platform_to_camera" type="fixed">
-    <parent link="base_link"/>
-    <child link="camera_link"/>
-    <origin xyz="0.15 0.0 0.3" rpy="0 0 0"/>
-  </joint>
-  <!-- ==================== Gazebo Plugins ==================== -->
-  <gazebo>
-    <plugin name="pumas_base_controller" filename="libgazebo_ros_planar_move.so">
-      <commandTopic>cmd_vel</commandTopic>
-      <odometryTopic>odom</odometryTopic>
-      <odometryFrame>odom</odometryFrame>
-      <odometryRate>50</odometryRate>
-      <robotBaseFrame>base_link</robotBaseFrame>
-    </plugin>
-  </gazebo>
-  <!-- ==================== Arm Manipulator (xArm) ==================== -->
-  <xacro:xarm_device prefix="xarm" hw_ns="xarm" dof="6" robot_type="xarm" load_gazebo_plugin="true" />
-  <!-- ==================== Gazebo Plugins for the Arm ==================== -->
-  <gazebo reference="xarm_base_link">
-    <plugin name="gazebo_ros_control" filename="libgazebo_ros_control.so"/>
-  </gazebo>
-  <!-- ==================== Attach the Arm to the Platform ==================== -->
-<joint name="platform_to_xarm" type="fixed">
-  <parent link="platform_link"/>
-    <child link="xarmlink_base"/>  <!-- Corrected to match the arm's base link -->
-  <origin xyz="0 0 0.45" rpy="0 0 0"/>
-</joint>
 </robot>

Commit message: sim festeshi

File: src/Hardware/robotino/robotino_description/urdf/robotino_armful.urdf.xacro (robot description, xacro)
@@ -1,4 +1,7 @@
 <?xml version="1.0"?>
-<robot name="festoshi" xmlns:xacro="http://ros.org/wiki/xacro">
+<robot name="festeshi" xmlns:xacro="http://ros.org/wiki/xacro">
+<gazebo>
+  <static>false</static>
+</gazebo>
   <!-- ARGUMENTS -->
   <xacro:arg name="add_gripper" default="false"/>
@@ -10,27 +13,87 @@
   <xacro:arg name="add_d435i_links" default="false"/>
   <xacro:arg name="robot_sn" default=""/>
-  <xacro:arg name="namespace" default=""/>
+  <xacro:arg name="namespace" default="xarm"/>
+  <xacro:arg name="attach_to" default="platform_link"/>
+  <xacro:arg name="prefix" default="" />
+  <xacro:property name="kinect_mesh" value="package://robotino_description/meshes/sensors/kinect.dae"/>
   <!-- INCLUDE base first, which is a full robot -->
   <xacro:include filename="$(find robotino_description)/urdf/robotino_armless.urdf.xacro"/>
-  <!-- INCLUDE arm, which defines a macro -->
-  <xacro:include filename="$(find xarm_description)/urdf/xarm_device.urdf.xacro"/>
-  <!-- Instantiate xarm_device directly -->
+<xacro:include filename="$(find xarm_description)/urdf/xarm_device_macro.xacro"/>
+  <!-- Instantiate xarm_device manually with control -->
   <xacro:xarm_device
     robot_type="xarm"
     dof="5"
+    prefix="$(arg prefix)"
     add_gripper="$(arg add_gripper)"
     add_vacuum_gripper="$(arg add_vacuum_gripper)"
-    effort_control="$(arg effort_control)"
-    velocity_control="$(arg xarm_velocity_control)"
+    effort_control="false"
+    velocity_control="false"
     model1300="$(arg model1300)"
     add_realsense_d435i="$(arg add_realsense_d435i)"
     add_d435i_links="$(arg add_d435i_links)"
     robot_sn="$(arg robot_sn)"
-    hw_ns="$(arg namespace)" />
-  <!-- Connect base and arm -->
-  <joint name="xarm_mount" type="fixed">
-    <parent link="base_link"/>
-    <child link="link_base"/>
-    <origin xyz="0 0 0.75" rpy="0 0 0"/>
-  </joint>
+    hw_ns="$(arg namespace)"
+    attach_to="$(arg attach_to)"
+    create_attach_link="false" />
+<!-- === Kinect mounted on link5 === -->
+<!-- Fixed joint that attaches the Kinect to the arm -->
+<joint name="camera_joint" type="fixed">
+  <parent link="link5"/>
+  <child  link="camera_link"/>
+  <!-- tweak xyz/rpy to match the real mounting position -->
+  <origin xyz="0.0 0 0.0" rpy="0 0 0"/>
+</joint>
+<!-- Kinect link body -->
+<link name="camera_link">
+  <visual>
+  <origin xyz="0.08 0.0 -0.04" rpy="-1.57 0 -1.57"/>
+    <geometry>
+      <mesh filename="${kinect_mesh}" scale="1 1 1"/>
+    </geometry>
+  </visual>
+  <collision>
+  <origin xyz="0.08 0.0 -0.04" rpy="-1.57 0 -1.57"/>
+    <geometry>
+      <mesh filename="${kinect_mesh}" scale="1 1 1"/>
+    </geometry>
+  </collision>
+</link>
+<!-- Gazebo depth-camera sensor plugin -->
+<gazebo reference="camera_link">
+ <sensor type="depth" name="kinect_sensor">
+<pose>0 0 0 -1.5708 -1.5708 -1.5708</pose>
+  <always_on>true</always_on>
+  <update_rate>30</update_rate>
+  <visualize>true</visualize>
+  <camera>
+    <horizontal_fov>1.0472</horizontal_fov> <!-- 60 deg -->
+    <image>
+      <width>640</width>
+      <height>480</height>
+      <format>R8G8B8</format>
+    </image>
+    <depth_near>0.1</depth_near>
+    <depth_far>10.0</depth_far>
+  </camera>
+  <plugin name="kinect_controller" filename="libgazebo_ros_openni_kinect.so">
+    <alwaysOn>true</alwaysOn>
+    <updateRate>30.0</updateRate>
+    <cameraName>camera</cameraName>
+    <imageTopicName>rgb/image_raw</imageTopicName>
+    <depthImageTopicName>depth/image_raw</depthImageTopicName>
+    <depthImageCameraInfoTopicName>depth/camera_info</depthImageCameraInfoTopicName>
+    <pointCloudTopicName>depth_registered/points</pointCloudTopicName>
+    <frameName>camera_link</frameName>
+    <hackBaseline>0.07</hackBaseline>
+    <depthImageFormat>16UC1</depthImageFormat>
+    <imageFormat>R8G8B8</imageFormat>
+    <distortionK1>0.0</distortionK1>
+    <distortionK2>0.0</distortionK2>
+    <distortionK3>0.0</distortionK3>
+    <distortionT1>0.0</distortionT1>
+    <distortionT2>0.0</distortionT2>
+  </plugin>
+</sensor>
+</gazebo>
+<!-- === End Kinect block === -->
 </robot>

File: src/Hardware/robotino/robotino_description/urdf/robotino_armless.urdf.xacro (robot description, xacro)
@@ -15,5 +15,4 @@
   <xacro:property name="tower_mesh" value="package://robotino_description/model/Robotino3_Platform-xarm.dae"/>
   <xacro:property name="hokuyo_mesh" value="package://robotino_description/meshes/sensors/hokuyo.dae"/>
-  <xacro:property name="kinect_mesh" value="package://robotino_description/meshes/sensors/kinect.dae"/>
   <!-- ==================== Macros ==================== -->
   <xacro:macro name="wheel_link" params="index xyz rpy">
@@ -48,5 +47,5 @@
     <inertial>
       <origin xyz="0 0 0.03" rpy="0 0 0"/>
-      <mass value="35.0"/>
+      <mass value="55.0"/>
       <inertia ixx="1.0" iyy="1.0" izz="1.0" ixy="0.0" ixz="0.0" iyz="0.0"/>
     </inertial>
@@ -114,24 +113,4 @@
     <origin xyz="0.07 0.0 0.28" rpy="0 0 0"/>
   </joint>
-  <!-- ==================== Kinect Sensor ==================== -->
-  <link name="camera_link">
-    <visual>
-      <origin xyz="0.15 0 0" rpy="0 0 1.57"/>
-      <geometry>
-        <mesh filename="${kinect_mesh}" scale="1 1 1"/>
-      </geometry>
-    </visual>
-    <collision>
-      <origin xyz="0.15 0 0" rpy="0 0 1.57"/>
-      <geometry>
-        <mesh filename="${kinect_mesh}" scale="1 1 1"/>
-      </geometry>
-    </collision>
-  </link>
-  <joint name="platform_to_camera" type="fixed">
-    <parent link="base_link"/>
-    <child link="camera_link"/>
-    <origin xyz="0.15 0.0 0.3" rpy="0 0 0"/>
-  </joint>
   <!-- ==================== Gazebo Plugins ==================== -->
   <gazebo>
@@ -176,27 +155,7 @@
     </sensor>
   </gazebo>
-  <gazebo reference="camera_link">
-    <sensor type="depth" name="kinect_sensor">
-      <always_on>true</always_on>
-      <update_rate>30</update_rate>
-      <visualize>true</visualize>
-      <camera>
-        <horizontal_fov>1.0472</horizontal_fov>  <!-- 60° FOV -->
-        <image>
-          <width>640</width>
-          <height>480</height>
-          <format>R8G8B8</format>
-        </image>
-        <depth_near>0.1</depth_near>
-        <depth_far>10.0</depth_far>
-      </camera>
-      <plugin name="kinect_controller" filename="libgazebo_ros_openni_kinect.so">
-        <topicName>/kinect/depth</topicName>
-        <frameName>camera_link</frameName>
-        <baseline>0.1</baseline>
-        <alwaysOn>true</alwaysOn>
-        <updateRate>30</updateRate>
-      </plugin>
-    </sensor>
-  </gazebo>
+<gazebo>
+  <plugin name="gazebo_ros_control" filename="libgazebo_ros_control.so">
+    <robotNamespace>/xarm</robotNamespace>  </plugin>
+</gazebo>
 </robot>

Commit message: lets robocup

File: src/Hardware/robotino/robotino_description/urdf/robotino_armful.urdf.xacro (robot description, xacro)
@@ -46,4 +46,19 @@
 <!-- Kinect link body -->
 <link name="camera_link">
+  <!-- ✅ Standard ROS optical frame -->
+  <link name="camera_depth_optical_frame">
+  <visual>
+    <origin xyz="0 0 0" rpy="0 0 0"/>
+    <geometry>
+      <box size="0.01 0.01 0.01"/>
+    </geometry>
+    <material name="Grey"/>
+  </visual>
+</link>
+<joint name="camera_depth_optical_joint" type="fixed">
+    <parent link="camera_link"/>
+    <child link="camera_depth_optical_frame"/>
+    <origin xyz="0 0 0" rpy="-1.5708 0 -1.5708"/>
+  </joint>
   <visual>
   <origin xyz="0.08 0.0 -0.04" rpy="-1.57 0 -1.57"/>
